File: pcb/pyramid-of-brightness.kicad_pcb (KiCad board)
At the start: 2 copper layers, 99 x 99 mm, 290 parts, among them J3 USB_C_Receptacle_USB2.0_14P, J4 Conn_01x02, U1 BMP388, U2 ICM-42688-P, U3 TXB0108RGY, U4 W25Q128JVS, U5 NCP1117-3.3_SOT223, U6 RP2040, X2 ABM8-272-T3

Commit message: Finished board
Parts:
- added G***: LOGO, LOGO, B.Cu at (104.3, 96.4)
- added G***: LOGO, LOGO, B.Cu at (138.5, 91.0)
- added G***: LOGO, LOGO, B.Cu at (139.1, 65.5)
- added G***: LOGO, LOGO, B.Cu at (60.4, 49.7)
- moved U2 0.21 mm to (134.1, 43.2), turned to 90 degrees
Routing:
- net GYRO_INT2: track 0.00 -> 59.7 mm, vias 0 -> 2
- net SPI_MOSI: track 0.00 -> 58.9 mm, vias 0 -> 5
- net SPI_MISO: track 0.00 -> 57.4 mm, vias 0 -> 5
- net SPI_SCK: track 0.00 -> 57.1 mm, vias 0 -> 5
- net SPI_GYRO_CP: track 0.00 -> 54.5 mm
- net BARO_INT: track 0.00 -> 53.6 mm, vias 0 -> 4
- net SPI_BARO_CP: track 0.00 -> 51.6 mm, vias 0 -> 2
- net GYRO_INT: track 0.00 -> 48.8 mm
- net +5V: track 2114.8 -> 2073.8 mm, vias 0 -> 4
- net GND: track 0.22 -> 36.9 mm, vias 0 -> 128
- net +1V1: track 6.51 -> 25.9 mm, vias 0 -> 3
- net /USB D+: track 45.8 -> 57.0 mm
- net /USB D-: track 45.8 -> 55.5 mm, vias 2 -> 4
- net (no net): track 7.97 -> 0.00 mm, vias 2 -> 0
- net +3V3: track 134.1 -> 138.3 mm
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Other:
- board text added: "- Wilmer von Harpe -"
- board text added: "BOOT"
- board text added: "Pyramid of Brightness"
- board text added: "Rev 1, 21.4.2025"
